File: codec.kicad_sch (KiCad schematic)
At the start: 14 parts, among them J4 Conn_01x02, J5 AudioJack4, U3 TLV320AIC3100

Commit message: pcb: add audio layout
Connections:
- net HPL: now also C21.1, U3.27 (HPL); no longer C21.2, J5.T
- net HPR: now also C23.1, U3.30 (HPR); no longer C23.2, J5.R1
- new net: C23.2, J5.R1
- new net: C21.2, J5.T
Other:
- moved on the sheet: C21, C23
Changed lines of the file:
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@@
 	)
 	(junction
-		(at 176.53 105.41)
-		(diameter 0)
-		(color 0 0 0 0)
-	)
-	(junction
 		(at 147.32 127)
 		(diameter 0)
@@
 	)
 	(junction
-		(at 176.53 102.87)
+		(at 167.64 105.41)
+		(diameter 0)
+		(color 0 0 0 0)
+	)
+	(junction
+		(at 167.64 102.87)
 		(diameter 0)
 		(color 0 0 0 0)
@@
 	(wire
 		(pts
-			(xy 176.53 105.41) (xy 184.15 105.41)
+			(xy 181.61 105.41) (xy 184.15 105.41)
 		)
 		(stroke
@@
 	(wire
 		(pts
-			(xy 167.64 102.87) (xy 168.91 102.87)
+			(xy 167.64 102.87) (xy 173.99 102.87)
 		)
 		(stroke
@@
 	(wire
 		(pts
-			(xy 176.53 101.6) (xy 176.53 102.87)
+			(xy 167.64 106.68) (xy 167.64 105.41)
 		)
 		(stroke
@@
 	(wire
 		(pts
+			(xy 168.91 106.68) (xy 167.64 106.68)
+		)
+		(stroke
+			(width 0)
+			(type default)
+		)
+	)
+	(wire
+		(pts
 			(xy 149.86 82.55) (xy 149.86 85.09)
 		)
@@
 	(wire
 		(pts
-			(xy 176.53 102.87) (xy 184.15 102.87)
+			(xy 179.07 102.87) (xy 184.15 102.87)
 		)
 		(stroke
@@
 	(wire
 		(pts
-			(xy 173.99 102.87) (xy 176.53 102.87)
-		)
-		(stroke
-			(width 0)
-			(type default)
-		)
-	)
-	(wire
-		(pts
 			(xy 151.13 72.39) (xy 151.13 82.55)
 		)
@@
 	(wire
 		(pts
-			(xy 176.53 106.68) (xy 176.53 105.41)
+			(xy 167.64 101.6) (xy 168.91 101.6)
 		)
 		(stroke
@@
 	(wire
 		(pts
-			(xy 167.64 105.41) (xy 171.45 105.41)
+			(xy 167.64 105.41) (xy 176.53 105.41)
 		)
 		(stroke
@@
 	(wire
 		(pts
-			(xy 177.8 106.68) (xy 176.53 106.68)
-		)
-		(stroke
-			(width 0)
-			(type default)
-		)
-	)
-	(wire
-		(pts
-			(xy 176.53 101.6) (xy 177.8 101.6)
+			(xy 139.7 127) (xy 142.24 127)
 		)
 		(stroke
@@
 	(wire
 		(pts
-			(xy 139.7 127) (xy 142.24 127)
+			(xy 123.19 110.49) (xy 127 110.49)
 		)
 		(stroke
@@
 	(wire
 		(pts
-			(xy 123.19 110.49) (xy 127 110.49)
+			(xy 167.64 115.57) (xy 168.91 115.57)
 		)
 		(stroke
@@
 	(wire
 		(pts
-			(xy 167.64 115.57) (xy 168.91 115.57)
+			(xy 170.18 91.44) (xy 172.72 91.44)
 		)
 		(stroke
@@
 	(wire
 		(pts
-			(xy 170.18 91.44) (xy 172.72 91.44)
+			(xy 152.4 125.73) (xy 152.4 127)
 		)
 		(stroke
@@
 	(wire
 		(pts
-			(xy 152.4 125.73) (xy 152.4 127)
+			(xy 167.64 101.6) (xy 167.64 102.87)
 		)
 		(stroke
@@
 		)
 	)
+	(hierarchical_label "HPR"
+		(shape output)
+		(at 168.91 106.68 0)
+		(effects
+			(font
+				(size 1.27 1.27)
+			)
+			(justify left)
+		)
+	)
 	(hierarchical_label "MCLK"
 		(shape input)
@@
 		)
 	)
-	(hierarchical_label "SDA"
-		(shape bidirectional)
-		(at 123.19 97.79 180)
+	(hierarchical_label "HPL"
+		(shape output)
+		(at 168.91 101.6 0)
 		(effects
 			(font
 				(size 1.27 1.27)
 			)
-			(justify right)
+			(justify left)
 		)
 	)
-	(hierarchical_label "HPL"
-		(shape output)
-		(at 177.8 101.6 0)
+	(hierarchical_label "SDA"
+		(shape bidirectional)
+		(at 123.19 97.79 180)
 		(effects
 			(font
 				(size 1.27 1.27)
 			)
-			(justify left)
+			(justify right)
 		)
 	)
@@
 		)
 	)
-	(hierarchical_label "HPR"
-		(shape output)
-		(at 177.8 106.68 0)
-		(effects
-			(font
-				(size 1.27 1.27)
-			)
-			(justify left)
-		)
-	)
 	(hierarchical_label "DIN"
 		(shape input)
@@
 	(symbol
 		(lib_id "Device:C_Small")
-		(at 173.99 105.41 90)
+		(at 179.07 105.41 90)
 		(unit 1)
 		(body_style 1)
@@
 		(dnp no)
 		(property "Reference" "C23"
-			(at 171.45 106.934 90)
+			(at 176.53 106.934 90)
 			(show_name no)
 			(do_not_autoplace no)
@@
 		)
 		(property "Value" "10u"
-			(at 171.45 108.712 90)
+			(at 176.53 108.712 90)
 			(show_name no)
 			(do_not_autoplace no)
@@
 		)
 		(property "Footprint" "Capacitor_SMD:C_0805_2012Metric"
-			(at 173.99 105.41 0)
+			(at 179.07 105.41 0)
 			(hide yes)
 			(show_name no)
@@
 		)
 		(property "Datasheet" ""
-			(at 173.99 105.41 0)
+			(at 179.07 105.41 0)
 			(hide yes)
 			(show_name no)
@@
 		)
 		(property "Description" "Unpolarized capacitor, small symbol"
-			(at 173.99 105.41 0)
+			(at 179.07 105.41 0)
 			(hide yes)
 			(show_name no)
@@
 		)
 		(property "Manufacturer" "Murata"
-			(at 173.99 105.41 0)
+			(at 179.07 105.41 0)
 			(hide yes)
 			(show_name no)
@@
 		)
 		(property "Manufacturer Part Number" "GRM21BR61H106KE43L"
-			(at 173.99 105.41 0)
+			(at 179.07 105.41 0)
 			(hide yes)
 			(show_name no)
@@
 		)
 		(property "Basic" "Y"
-			(at 173.99 105.41 0)
+			(at 179.07 105.41 0)
 			(hide yes)
 			(show_name no)
@@
 		)
 		(property "JLCPCB Part #" "C440198"
-			(at 173.99 105.41 0)
+			(at 179.07 105.41 0)
 			(hide yes)
 			(show_name no)
@@
 	(symbol
 		(lib_id "Device:C_Small")
-		(at 171.45 102.87 90)
+		(at 176.53 102.87 90)
 		(unit 1)
 		(body_style 1)
@@
 		(dnp no)
 		(property "Reference" "C21"
-			(at 169.672 97.79 90)
+			(at 179.578 99.568 90)
 			(show_name no)
 			(do_not_autoplace no)
@@
 		)
 		(property "Value" "10u"
-			(at 169.672 99.568 90)
+			(at 179.578 101.346 90)
 			(show_name no)
 			(do_not_autoplace no)
@@
 		)
 		(property "Footprint" "Capacitor_SMD:C_0805_2012Metric"
-			(at 171.45 102.87 0)
+			(at 176.53 102.87 0)
 			(hide yes)
 			(show_name no)
@@
 		)
 		(property "Datasheet" ""
-			(at 171.45 102.87 0)
+			(at 176.53 102.87 0)
 			(hide yes)
 			(show_name no)
@@
 		)
 		(property "Description" "Unpolarized capacitor, small symbol"
-			(at 171.45 102.87 0)
+			(at 176.53 102.87 0)
 			(hide yes)
 			(show_name no)
@@
 		)
 		(property "Manufacturer" "Murata"
-			(at 171.45 102.87 0)
+			(at 176.53 102.87 0)
 			(hide yes)
 			(show_name no)
@@
 		)
 		(property "Manufacturer Part Number" "GRM21BR61H106KE43L"
-			(at 171.45 102.87 0)
+			(at 176.53 102.87 0)
 			(hide yes)
 			(show_name no)
@@
 		)
 		(property "Basic" "Y"
-			(at 171.45 102.87 0)
+			(at 176.53 102.87 0)
 			(hide yes)
 			(show_name no)
@@
 		)
 		(property "JLCPCB Part #" "C440198"
-			(at 171.45 102.87 0)
+			(at 176.53 102.87 0)
 			(hide yes)
 			(show_name no)
