File: codec.kicad_sch (KiCad schematic)
At the start: 14 parts, among them J4 Conn_01x02, J5 AudioJack4, U3 TLV320AIC3100

Commit message: pcb(silk): add user txt
Other:
- note added: "2.5W"
- note removed: "4W"
Changed lines of the file:
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@@
 		(company "Rémi Ait-Younes")
 	)
-	(text "4W"
+	(text "2.5W"
 		(exclude_from_sim no)
 		(at 176.53 97.282 0)

Commit message: generate production files
Parts:
- J5: JLCPCB Part # C431535 -> C521460; Manufacturer Shou HAN -> USAKRO
Changed lines of the file:
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@@
 			)
 		)
-		(property "JLCPCB Part #" "C431535"
+		(property "JLCPCB Part #" "C521460"
 			(at 189.23 107.95 0)
 			(hide yes)
@@
 			)
 		)
-		(property "Manufacturer" "Shou HAN"
+		(property "Manufacturer" "USAKRO"
 			(at 189.23 107.95 0)
 			(hide yes)
